File: hardware/output/kicad/xiao_voice_recorder.kicad_sch (KiCad schematic)
At the start: 63 parts, among them J1 TYPE-C-16P, J2 JST-PH-2P-LiPo, Q1 AO3401A_P-FET, SW1 POWER_SWITCH, SW2 RESET_BTN, SW3 BOOT_BTN, U1 USBLC6-2SC6, U2 TP4056, U3 AP2112K-3.3, U4 ESP32-C3-WROOM-02-N4, U5 LSM6DS3TR-C, U6 W25Q128JV_16MB

Commit message: fix(hardware): resolve inherited ancestor symbols in schematic to fix KiCad loading error
Changed lines of the file:
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@@
   (wire (pts (xy 35.00 71.81) (xy 35.00 76.89)) (stroke (width 0) (type default)))
   (label "GND" (at 35.00 76.89 270) (fields_autoplaced yes) (effects (font (size 1.27 1.27)) (justify right)))
-  (wire (pts (xy 77.00 64.19) (xy 77.00 59.11)) (stroke (width 0) (type default)))
-  (label "USB_DP" (at 77.00 59.11 90) (fields_autoplaced yes) (effects (font (size 1.27 1.27)) (justify left)))
-  (wire (pts (xy 77.00 71.81) (xy 77.00 76.89)) (stroke (width 0) (type default)))
-  (label "GND" (at 77.00 76.89 270) (fields_autoplaced yes) (effects (font (size 1.27 1.27)) (justify right)))
-  (wire (pts (xy 77.00 71.81) (xy 77.00 76.89)) (stroke (width 0) (type default)))
-  (label "USB_DN" (at 77.00 76.89 270) (fields_autoplaced yes) (effects (font (size 1.27 1.27)) (justify right)))
-  (wire (pts (xy 77.00 71.81) (xy 77.00 76.89)) (stroke (width 0) (type default)))
-  (label "USB_DN" (at 77.00 76.89 270) (fields_autoplaced yes) (effects (font (size 1.27 1.27)) (justify right)))
-  (wire (pts (xy 77.00 71.81) (xy 77.00 76.89)) (stroke (width 0) (type default)))
-  (label "VBUS" (at 77.00 76.89 270) (fields_autoplaced yes) (effects (font (size 1.27 1.27)) (justify right)))
-  (wire (pts (xy 77.00 71.81) (xy 77.00 76.89)) (stroke (width 0) (type default)))
-  (label "USB_DP" (at 77.00 76.89 270) (fields_autoplaced yes) (effects (font (size 1.27 1.27)) (justify right)))
+  (wire (pts (xy 71.92 68.00) (xy 66.84 68.00)) (stroke (width 0) (type default)))
+  (label "USB_DP" (at 66.84 68.00 180) (fields_autoplaced yes) (effects (font (size 1.27 1.27)) (justify right)))
+  (wire (pts (xy 77.00 75.62) (xy 77.00 80.70)) (stroke (width 0) (type default)))
+  (label "GND" (at 77.00 80.70 270) (fields_autoplaced yes) (effects (font (size 1.27 1.27)) (justify right)))
+  (wire (pts (xy 71.92 70.54) (xy 66.84 70.54)) (stroke (width 0) (type default)))
+  (label "USB_DN" (at 66.84 70.54 180) (fields_autoplaced yes) (effects (font (size 1.27 1.27)) (justify right)))
+  (wire (pts (xy 82.08 70.54) (xy 87.16 70.54)) (stroke (width 0) (type default)))
+  (label "USB_DN" (at 87.16 70.54 0) (fields_autoplaced yes) (effects (font (size 1.27 1.27)) (justify left)))
+  (wire (pts (xy 77.00 62.92) (xy 77.00 57.84)) (stroke (width 0) (type default)))
+  (label "VBUS" (at 77.00 57.84 90) (fields_autoplaced yes) (effects (font (size 1.27 1.27)) (justify left)))
+  (wire (pts (xy 82.08 68.00) (xy 87.16 68.00)) (stroke (width 0) (type default)))
+  (label "USB_DP" (at 87.16 68.00 0) (fields_autoplaced yes) (effects (font (size 1.27 1.27)) (justify left)))
   (wire (pts (xy 119.00 64.19) (xy 119.00 59.11)) (stroke (width 0) (type default)))
   (label "GND" (at 119.00 59.11 90) (fields_autoplaced yes) (effects (font (size 1.27 1.27)) (justify left)))
@@
   (wire (pts (xy 155.92 124.00) (xy 150.84 124.00)) (stroke (width 0) (type default)))
   (label "VBAT" (at 150.84 124.00 180) (fields_autoplaced yes) (effects (font (size 1.27 1.27)) (justify right)))
-  (wire (pts (xy 35.00 148.19) (xy 35.00 143.11)) (stroke (width 0) (type default)))
-  (label "VBUS" (at 35.00 143.11 90) (fields_autoplaced yes) (effects (font (size 1.27 1.27)) (justify left)))
-  (wire (pts (xy 35.00 155.81) (xy 35.00 160.89)) (stroke (width 0) (type default)))
-  (label "VBAT" (at 35.00 160.89 270) (fields_autoplaced yes) (effects (font (size 1.27 1.27)) (justify right)))
-  (wire (pts (xy 35.00 155.81) (xy 35.00 160.89)) (stroke (width 0) (type default)))
-  (label "V_SYS" (at 35.00 160.89 270) (fields_autoplaced yes) (effects (font (size 1.27 1.27)) (justify right)))
+  (wire (pts (xy 29.92 152.00) (xy 24.84 152.00)) (stroke (width 0) (type default)))
+  (label "VBUS" (at 24.84 152.00 180) (fields_autoplaced yes) (effects (font (size 1.27 1.27)) (justify right)))
+  (wire (pts (xy 37.54 157.08) (xy 37.54 162.16)) (stroke (width 0) (type default)))
+  (label "VBAT" (at 37.54 162.16 270) (fields_autoplaced yes) (effects (font (size 1.27 1.27)) (justify right)))
+  (wire (pts (xy 37.54 146.92) (xy 37.54 141.84)) (stroke (width 0) (type default)))
+  (label "V_SYS" (at 37.54 141.84 90) (fields_autoplaced yes) (effects (font (size 1.27 1.27)) (justify left)))
   (wire (pts (xy 77.00 148.19) (xy 77.00 143.11)) (stroke (width 0) (type default)))
   (label "VBUS" (at 77.00 143.11 90) (fields_autoplaced yes) (effects (font (size 1.27 1.27)) (justify left)))
@@
   (wire (pts (xy 122.81 152.00) (xy 127.89 152.00)) (stroke (width 0) (type default)))
   (label "VBUS" (at 127.89 152.00 0) (fields_autoplaced yes) (effects (font (size 1.27 1.27)) (justify left)))
-  (wire (pts (xy 161.00 148.19) (xy 161.00 143.11)) (stroke (width 0) (type default)))
-  (label "V_SYS" (at 161.00 143.11 90) (fields_autoplaced yes) (effects (font (size 1.27 1.27)) (justify left)))
-  (wire (pts (xy 161.00 155.81) (xy 161.00 160.89)) (stroke (width 0) (type default)))
-  (label "GND" (at 161.00 160.89 270) (fields_autoplaced yes) (effects (font (size 1.27 1.27)) (justify right)))
-  (wire (pts (xy 161.00 155.81) (xy 161.00 160.89)) (stroke (width 0) (type default)))
-  (label "V_SYS" (at 161.00 160.89 270) (fields_autoplaced yes) (effects (font (size 1.27 1.27)) (justify right)))
-  (wire (pts (xy 161.00 155.81) (xy 161.00 160.89)) (stroke (width 0) (type default)))
-  (label "+3V3" (at 161.00 160.89 270) (fields_autoplaced yes) (effects (font (size 1.27 1.27)) (justify right)))
+  (wire (pts (xy 153.38 149.46) (xy 148.30 149.46)) (stroke (width 0) (type default)))
+  (label "V_SYS" (at 148.30 149.46 180) (fields_autoplaced yes) (effects (font (size 1.27 1.27)) (justify right)))
+  (wire (pts (xy 161.00 159.62) (xy 161.00 164.70)) (stroke (width 0) (type default)))
+  (label "GND" (at 161.00 164.70 270) (fields_autoplaced yes) (effects (font (size 1.27 1.27)) (justify right)))
+  (wire (pts (xy 153.38 152.00) (xy 148.30 152.00)) (stroke (width 0) (type default)))
+  (label "V_SYS" (at 148.30 152.00 180) (fields_autoplaced yes) (effects (font (size 1.27 1.27)) (justify right)))
+  (wire (pts (xy 168.62 149.46) (xy 173.70 149.46)) (stroke (width 0) (type default)))
+  (label "+3V3" (at 173.70 149.46 0) (fields_autoplaced yes) (effects (font (size 1.27 1.27)) (justify left)))
   (wire (pts (xy 35.00 176.19) (xy 35.00 171.11)) (stroke (width 0) (type default)))
   (label "V_SYS" (at 35.00 171.11 90) (fields_autoplaced yes) (effects (font (size 1.27 1.27)) (justify left)))
@@
   (wire (pts (xy 255.00 178.81) (xy 255.00 183.89)) (stroke (width 0) (type default)))
   (label "GND" (at 255.00 183.89 270) (fields_autoplaced yes) (effects (font (size 1.27 1.27)) (justify right)))
-  (wire (pts (xy 291.00 171.19) (xy 291.00 166.11)) (stroke (width 0) (type default)))
-  (label "SPI_CS" (at 291.00 166.11 90) (fields_autoplaced yes) (effects (font (size 1.27 1.27)) (justify left)))
-  (wire (pts (xy 291.00 178.81) (xy 291.00 183.89)) (stroke (width 0) (type default)))
-  (label "SPI_MISO" (at 291.00 183.89 270) (fields_autoplaced yes) (effects (font (size 1.27 1.27)) (justify right)))
-  (wire (pts (xy 291.00 178.81) (xy 291.00 183.89)) (stroke (width 0) (type default)))
-  (label "GND" (at 291.00 183.89 270) (fields_autoplaced yes) (effects (font (size 1.27 1.27)) (justify right)))
-  (wire (pts (xy 291.00 178.81) (xy 291.00 183.89)) (stroke (width 0) (type default)))
-  (label "SPI_MOSI" (at 291.00 183.89 270) (fields_autoplaced yes) (effects (font (size 1.27 1.27)) (justify right)))
-  (wire (pts (xy 291.00 178.81) (xy 291.00 183.89)) (stroke (width 0) (type default)))
-  (label "SPI_CLK" (at 291.00 183.89 270) (fields_autoplaced yes) (effects (font (size 1.27 1.27)) (justify right)))
-  (wire (pts (xy 291.00 178.81) (xy 291.00 183.89)) (stroke (width 0) (type default)))
-  (label "+3V3" (at 291.00 183.89 270) (fields_autoplaced yes) (effects (font (size 1.27 1.27)) (justify right)))
+  (wire (pts (xy 280.84 167.38) (xy 275.76 167.38)) (stroke (width 0) (type default)))
+  (label "SPI_CS" (at 275.76 167.38 180) (fields_autoplaced yes) (effects (font (size 1.27 1.27)) (justify right)))
+  (wire (pts (xy 280.84 175.00) (xy 275.76 175.00)) (stroke (width 0) (type default)))
+  (label "SPI_MISO" (at 275.76 175.00 180) (fields_autoplaced yes) (effects (font (size 1.27 1.27)) (justify right)))
+  (wire (pts (xy 291.00 187.70) (xy 291.00 192.78)) (stroke (width 0) (type default)))
+  (label "GND" (at 291.00 192.78 270) (fields_autoplaced yes) (effects (font (size 1.27 1.27)) (justify right)))
+  (wire (pts (xy 280.84 172.46) (xy 275.76 172.46)) (stroke (width 0) (type default)))
+  (label "SPI_MOSI" (at 275.76 172.46 180) (fields_autoplaced yes) (effects (font (size 1.27 1.27)) (justify right)))
+  (wire (pts (xy 280.84 169.92) (xy 275.76 169.92)) (stroke (width 0) (type default)))
+  (label "SPI_CLK" (at 275.76 169.92 180) (fields_autoplaced yes) (effects (font (size 1.27 1.27)) (justify right)))
+  (wire (pts (xy 291.00 162.30) (xy 291.00 157.22)) (stroke (width 0) (type default)))
+  (label "+3V3" (at 291.00 157.22 90) (fields_autoplaced yes) (effects (font (size 1.27 1.27)) (justify left)))
   (wire (pts (xy 255.00 199.19) (xy 255.00 194.11)) (stroke (width 0) (type default)))
   (label "+3V3" (at 255.00 194.11 90) (fields_autoplaced yes) (effects (font (size 1.27 1.27)) (justify left)))

Commit message: fix(hardware): fully flatten all extended symbols to eliminate KiCad parent loading errors
Connections:
- net +3V3: now also C1.2, C10.2, C11.1, C11.2, C12.1, C12.2, C13.1, C13.2, C14.1, C14.2, C15.1, C15.2, C16.1, C16.2, C17.1, C17.2, C18.1, C18.2, C2.1, C2.2, C3.1, C3.2, C4.1, C4.2, C5.1, C5.2, C6.1, C6.2, C7.1, C7.2, C8.1, C8.2, C9.1, C9.2, D3.1 (K), D3.2 (A), D4.1 (K), D5.1 (K), FB1.1, FB1.2, Q1.1 (G), Q1.3 (D), R1.2, R10.1, R11.1, R12.1, R12.2, R13.1, R13.2, R14.1, R14.2, R15.1, R16.1, R17.1, R18.1, R2.2, R3.2, R4.2, R5.1, R6.1, R7.1, R7.2, R8.2, R9.1, R9.2, SW1.1 (A), SW2.2, SW3.2, TP1.1, TP2.1, TP3.1, TP4.1, TP5.1, TP6.1, U1.1 (I/O1), U1.2 (GND), U1.3 (I/O2), U1.4 (I/O2), U1.5 (VBUS), U1.6 (I/O1), U3.1 (VIN), U3.2 (GND), U3.3 (EN), U3.5 (VOUT), U5.1 (SDO/SA0), U5.12 (CS), U5.13 (SCL), U5.14 (SDA), U5.4 (INT1), U5.5 (VDDIO), U5.6 (GND), U5.7 (GND), U5.8 (VDD), U6.1 (~{CS}), U6.2 (DO(IO1)), U6.4 (GND), U6.5 (DI(IO0)), U6.6 (CLK), U6.8 (VCC)
- net VBAT: now also Q1.2 (S), R8.1, SW1.2 (B), TP7.1

Commit message: fix(hardware): extract clean short library names from SKiDL objects for KiCad 8 schematic symbols
Parts:
- removed C1: 4.7nF_1kV, Capacitor_SMD:C_0805_2012Metric, symbol Ammeter_AC: AC ammeter Ammeter_DC: DC ammeter Antenna: Antenna Antenna_Chip: Ce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
- removed C10, C15: 1uF, Capacitor_SMD:C_0603_1608Metric, symbol Ammeter_AC: AC ammeter Ammeter_DC: DC ammeter Antenna: Antenna Antenna_Chip: Ce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
- removed C11, C2, C3, C4, C5, C8: 10uF, Capacitor_SMD:C_0805_2012Metric, symbol Ammeter_AC: AC ammeter Ammeter_DC: DC ammeter Antenna: Antenna Antenna_Chip: Ce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
- removed C12, C13, C14, C16, C17, C18, C6, C7, C9: 100nF, Capacitor_SMD:C_0603_1608Metric, symbol Ammeter_AC: AC ammeter Ammeter_DC: DC ammeter Antenna: Antenna Antenna_Chip: Ce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
- removed D1: RED_CHRG, LED_SMD:LED_0603_1608Metric, symbol Ammeter_AC: AC ammeter Ammeter_DC: DC ammeter Antenna: Antenna Antenna_Chip: Ce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
- removed D2: GRN_FULL, LED_SMD:LED_0603_1608Metric, symbol Ammeter_AC: AC ammeter Ammeter_DC: DC ammeter Antenna: Antenna Antenna_Chip: Ce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
- removed D3: SS14_Schottky, Diode_SMD:D_SOD-123, symbol Ammeter_AC: AC ammeter Ammeter_DC: DC ammeter Antenna: Antenna Antenna_Chip: Ce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
- removed D4: RED_RECORDING, LED_SMD:LED_0805_2012Metric, symbol Ammeter_AC: AC ammeter Ammeter_DC: DC ammeter Antenna: Antenna Antenna_Chip: Ce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
- removed D5: BLU_3V3_PWR, LED_SMD:LED_0603_1608Metric, symbol Ammeter_AC: AC ammeter Ammeter_DC: DC ammeter Antenna: Antenna Antenna_Chip: Ce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
- removed FB1: 600R_100MHz, Resistor_SMD:R_0805_2012Metric, symbol Ammeter_AC: AC ammeter Ammeter_DC: DC ammeter Antenna: Antenna Antenna_Chip: Ce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
- removed J1: TYPE-C-16P, Connector_USB:USB_C_Receptacle_HRO_TYPE-C-31-M-12, symbol 4P2C: RJ connector, 4P2C (4 positions 2 connected) 4P2C_Shielded: RJ connector,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
- removed J2: JST-PH-2P-LiPo, Connector_JST:JST_PH_S2B-PH-K_1x02_P2.00mm_Horizontal, symbol 4P2C: RJ connector, 4P2C (4 positions 2 connected) 4P2C_Shielded: RJ connector,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
- removed MK1: INMP441_LEFT, Sensor_Audio:InvenSense_INMP441, symbol ESP32-C3-WROOM-02: Espressif ESP32-C3 Wi-Fi & BLE 5.0 Module, 4MB Flash, PCB An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
- removed MK2: INMP441_RIGHT, Sensor_Audio:InvenSense_INMP441, symbol ESP32-C3-WROOM-02: Espressif ESP32-C3 Wi-Fi & BLE 5.0 Module, 4MB Flash, PCB An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
- removed Q1: AO3401A_P-FET, Package_TO_SOT_SMD:SOT-23, symbol 2N7000: 0.2A Id, 200V Vds, N-Channel MOSFET, 2.6V Logic Level, TO-92 3SK263: 30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
- removed R1, R2: 5.1k_1%, Resistor_SMD:R_0603_1608Metric, symbol Ammeter_AC: AC ammeter Ammeter_DC: DC ammeter Antenna: Antenna Antenna_Chip: Ce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
- removed R10, R11, R14, R15, R16: 10k, Resistor_SMD:R_0603_1608Metric, symbol Ammeter_AC: AC ammeter Ammeter_DC: DC ammeter Antenna: Antenna Antenna_Chip: Ce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
- removed R12, R13: 4.7k, Resistor_SMD:R_0603_1608Metric, symbol Ammeter_AC: AC ammeter Ammeter_DC: DC ammeter Antenna: Antenna Antenna_Chip: Ce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
- removed R17: 330R, Resistor_SMD:R_0805_2012Metric, symbol Ammeter_AC: AC ammeter Ammeter_DC: DC ammeter Antenna: Antenna Antenna_Chip: Ce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
- removed R18, R5, R6: 1k, Resistor_SMD:R_0603_1608Metric, symbol Ammeter_AC: AC ammeter Ammeter_DC: DC ammeter Antenna: Antenna Antenna_Chip: Ce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
- removed R3: 1M, Resistor_SMD:R_0805_2012Metric, symbol Ammeter_AC: AC ammeter Ammeter_DC: DC ammeter Antenna: Antenna Antenna_Chip: Ce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
- removed R4: 2.4k_1%, Resistor_SMD:R_0603_1608Metric, symbol Ammeter_AC: AC ammeter Ammeter_DC: DC ammeter Antenna: Antenna Antenna_Chip: Ce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
- removed R7: 100k, Resistor_SMD:R_0603_1608Metric, symbol Ammeter_AC: AC ammeter Ammeter_DC: DC ammeter Antenna: Antenna Antenna_Chip: Ce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
- removed R8, R9: 100k_1%, Resistor_SMD:R_0603_1608Metric, symbol Ammeter_AC: AC ammeter Ammeter_DC: DC ammeter Antenna: Antenna Antenna_Chip: Ce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
- removed SW1: POWER_SWITCH, Button_Switch_SMD:SW_SPDT_PCM12, symbol SW_Coded: Rotary switch, 4-bit encoding SW_Coded_SH-7010: Rotary switch, 4-bit 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
- removed SW2: RESET_BTN, Button_Switch_SMD:SW_SPST_PTS645, symbol SW_Coded: Rotary switch, 4-bit encoding SW_Coded_SH-7010: Rotary switch, 4-bit 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
- removed SW3: BOOT_BTN, Button_Switch_SMD:SW_SPST_PTS645, symbol SW_Coded: Rotary switch, 4-bit encoding SW_Coded_SH-7010: Rotary switch, 4-bit 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
- removed TP1: TP_3V3, TestPoint:TestPoint_Pad_D1.0mm_OD2.0mm, symbol 4P2C: RJ connector, 4P2C (4 positions 2 connected) 4P2C_Shielded: RJ connector,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
- removed TP2: TP_GND, TestPoint:TestPoint_Pad_D1.0mm_OD2.0mm, symbol 4P2C: RJ connector, 4P2C (4 positions 2 connected) 4P2C_Shielded: RJ connector,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
- removed TP3: TP_EN, TestPoint:TestPoint_Pad_D1.0mm_OD2.0mm, symbol 4P2C: RJ connector, 4P2C (4 positions 2 connected) 4P2C_Shielded: RJ connector,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
- removed TP4: TP_IO9, TestPoint:TestPoint_Pad_D1.0mm_OD2.0mm, symbol 4P2C: RJ connector, 4P2C (4 positions 2 connected) 4P2C_Shielded: RJ connector,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
- removed TP5: TP_USB_DP, TestPoint:TestPoint_Pad_D1.0mm_OD2.0mm, symbol 4P2C: RJ connector, 4P2C (4 positions 2 connected) 4P2C_Shielded: RJ connector,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
- removed TP6: TP_USB_DN, TestPoint:TestPoint_Pad_D1.0mm_OD2.0mm, symbol 4P2C: RJ connector, 4P2C (4 positions 2 connected) 4P2C_Shielded: RJ connector,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
- removed TP7: TP_VBAT, TestPoint:TestPoint_Pad_D1.0mm_OD2.0mm, symbol 4P2C: RJ connector, 4P2C (4 positions 2 connected) 4P2C_Shielded: RJ connector,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
- removed U1: USBLC6-2SC6, Package_TO_SOT_SMD:SOT-23-6, symbol CDNBS08-SLVU2.8-4: Quad bidirectional transil, Suppressor for ESD protection, 5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
- removed U2: TP4056, Package_SO:SOP-8-PP_3.9x4.9mm_P1.27mm_EP, symbol ESP32-C3-WROOM-02: Espressif ESP32-C3 Wi-Fi & BLE 5.0 Module, 4MB Flash, PCB An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
- removed U3: AP2112K-3.3, Package_TO_SOT_SMD:SOT-23-5, symbol ADP3336ARMZ: High Accuracy Ultralow IQ, 500mA anyCAP Adjustable Low Dropout Reg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
- removed U4: ESP32-C3-WROOM-02-N4, RF_Module:ESP32-C3-WROOM-02, symbol ESP32-C3-WROOM-02: Espressif ESP32-C3 Wi-Fi & BLE 5.0 Module, 4MB Flash, PCB An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
- removed U5: LSM6DS3TR-C, Package_LGA:LGA-14_3x2.5mm_P0.5mm_LayoutBorder1x6y, symbol ADXL343: 3-Axis MEMS Accelerometer, 2/4/8/16g range, I2C/SPI, LGA-14 ADXL363: M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
- removed U6: W25Q128JV_16MB, Package_SO:SOIC-8_5.23x5.23mm_P1.27mm, symbol 28F400: PA28F400BX-T/B Flash EEProm 4-MBIT (256Kx16bits, 512Kx8bits) 5V, 12V Pr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
- added C1: 4.7nF_1kV, Capacitor_SMD:C_0805_2012Metric, symbol Device:C
- added C10, C15: 1uF, Capacitor_SMD:C_0603_1608Metric, symbol Device:C
- added C11, C2, C3, C4, C5, C8: 10uF, Capacitor_SMD:C_0805_2012Metric, symbol Device:C
- added C12, C13, C14, C16, C17, C18, C6, C7, C9: 100nF, Capacitor_SMD:C_0603_1608Metric, symbol Device:C
- added D1: RED_CHRG, LED_SMD:LED_0603_1608Metric, symbol Device:LED
- added D2: GRN_FULL, LED_SMD:LED_0603_1608Metric, symbol Device:LED
- added D3: SS14_Schottky, Diode_SMD:D_SOD-123, symbol Device:D_Schottky
- added D4: RED_RECORDING, LED_SMD:LED_0805_2012Metric, symbol Device:LED
- added D5: BLU_3V3_PWR, LED_SMD:LED_0603_1608Metric, symbol Device:LED
- added FB1: 600R_100MHz, Resistor_SMD:R_0805_2012Metric, symbol Device:FerriteBead
- added J1: TYPE-C-16P, Connector_USB:USB_C_Receptacle_HRO_TYPE-C-31-M-12, symbol Connector:USB_C_Receptacle_USB2.0_16P
- added J2: JST-PH-2P-LiPo, Connector_JST:JST_PH_S2B-PH-K_1x02_P2.00mm_Horizontal, symbol Connector:Conn_01x02_Pin
- added MK1: INMP441_LEFT, Sensor_Audio:InvenSense_INMP441, symbol Project_Symbols:INMP441
- added MK2: INMP441_RIGHT, Sensor_Audio:InvenSense_INMP441, symbol Project_Symbols:INMP441
- added Q1: AO3401A_P-FET, Package_TO_SOT_SMD:SOT-23, symbol Transistor_FET:AO3401A
- added R1, R2: 5.1k_1%, Resistor_SMD:R_0603_1608Metric, symbol Device:R
- added R10, R11, R14, R15, R16: 10k, Resistor_SMD:R_0603_1608Metric, symbol Device:R
- added R12, R13: 4.7k, Resistor_SMD:R_0603_1608Metric, symbol Device:R
- added R17: 330R, Resistor_SMD:R_0805_2012Metric, symbol Device:R
- added R18, R5, R6: 1k, Resistor_SMD:R_0603_1608Metric, symbol Device:R
- added R3: 1M, Resistor_SMD:R_0805_2012Metric, symbol Device:R
- added R4: 2.4k_1%, Resistor_SMD:R_0603_1608Metric, symbol Device:R
- added R7: 100k, Resistor_SMD:R_0603_1608Metric, symbol Device:R
- added R8, R9: 100k_1%, Resistor_SMD:R_0603_1608Metric, symbol Device:R
- added SW1: POWER_SWITCH, Button_Switch_SMD:SW_SPDT_PCM12, symbol Switch:SW_SPDT
- added SW2: RESET_BTN, Button_Switch_SMD:SW_SPST_PTS645, symbol Switch:SW_Push
- added SW3: BOOT_BTN, Button_Switch_SMD:SW_SPST_PTS645, symbol Switch:SW_Push
- added TP1: TP_3V3, TestPoint:TestPoint_Pad_D1.0mm_OD2.0mm, symbol Connector:TestPoint
- added TP2: TP_GND, TestPoint:TestPoint_Pad_D1.0mm_OD2.0mm, symbol Connector:TestPoint
- added TP3: TP_EN, TestPoint:TestPoint_Pad_D1.0mm_OD2.0mm, symbol Connector:TestPoint
- added TP4: TP_IO9, TestPoint:TestPoint_Pad_D1.0mm_OD2.0mm, symbol Connector:TestPoint
- added TP5: TP_USB_DP, TestPoint:TestPoint_Pad_D1.0mm_OD2.0mm, symbol Connector:TestPoint
- added TP6: TP_USB_DN, TestPoint:TestPoint_Pad_D1.0mm_OD2.0mm, symbol Connector:TestPoint
- added TP7: TP_VBAT, TestPoint:TestPoint_Pad_D1.0mm_OD2.0mm, symbol Connector:TestPoint
- added U1: USBLC6-2SC6, Package_TO_SOT_SMD:SOT-23-6, symbol Power_Protection:USBLC6-2SC6
- added U2: TP4056, Package_SO:SOP-8-PP_3.9x4.9mm_P1.27mm_EP, symbol Project_Symbols:TP4056
- added U3: AP2112K-3.3, Package_TO_SOT_SMD:SOT-23-5, symbol Regulator_Linear:AP2112K-3.3
- added U4: ESP32-C3-WROOM-02-N4, RF_Module:ESP32-C3-WROOM-02, symbol Project_Symbols:ESP32-C3-WROOM-02
- added U5: LSM6DS3TR-C, Package_LGA:LGA-14_3x2.5mm_P0.5mm_LayoutBorder1x6y, symbol Sensor_Motion:LSM6DS3
- added U6: W25Q128JV_16MB, Package_SO:SOIC-8_5.23x5.23mm_P1.27mm, symbol Memory_Flash:W25Q128JVS
Connections:
- net +3V3: now also C1.2, C10.2, C11.2, C12.2, C13.2, C14.2, C15.1, C15.2, C16.1, C16.2, C17.1, C17.2, C18.1, C18.2, C2.2, C3.2, C4.1, C4.2, C5.1, C5.2, C6.1, C6.2, C7.2, C8.1, C8.2, C9.1, C9.2, D3.1 (K), D4.1 (K), D5.1 (K), FB1.1, J1.A1 (GND), J1.A12 (GND), J1.B1 (GND), J1.B12 (GND), J2.2 (Pin_2), MK1.1 (L/R), MK1.2 (GND), MK2.2 (GND), Q1.3 (D), R1.2, R10.1, R11.1, R12.1, R13.1, R14.1, R15.1, R16.1, R18.1, R2.2, R3.2, R4.2, R7.2, R9.2, SW2.2, SW3.2, TP1.1, TP2.1, TP3.1, U1.2 (GND), U2.1 (TEMP), U2.3 (GND), U2.9 (EPAD), U3.1 (VIN), U3.2 (GND), U3.3 (EN), U3.5 (VOUT), U4.1 (GND), U4.10 (GND), U4.2 (3V3), U4.20 (GND), U4.21 (EPAD), U5.1 (SDO/SA0), U5.12 (CS), U5.5 (VDDIO), U5.6 (GND), U5.7 (GND), U5.8 (VDD), U6.4 (GND), U6.8 (VCC)
- net VBAT: now also Q1.2 (S), R8.1, SW1.2 (B), TP7.1
- new net +3V3_AUDIO: C11.1, C12.1, C13.1, C14.1, FB1.2, MK1.3 (VDD), MK2.1 (L/R), MK2.3 (VDD)
- new net BATT_SENSE: C7.1, R8.2, R9.1, U4.12 (IO0)
- new net I2C_SCL: R12.2, U4.7 (IO7), U5.13 (SCL)
- new net I2C_SDA: R13.2, U4.6 (IO6), U5.14 (SDA)
- new net I2S_SCK: MK1.5 (SCK), MK2.5 (SCK), U4.14 (IO2)
- new net I2S_SD: MK1.4 (SD), MK2.4 (SD), U4.4 (IO4)
- new net I2S_WS: MK1.6 (WS), MK2.6 (WS), U4.15 (IO3)
- new net IMU_INT: U4.13 (IO1), U5.4 (INT1)
- new net SPI_CLK: U4.8 (IO8), U6.6 (CLK)
- new net SPI_CS: R14.2, U4.5 (IO5), U6.1 (~{CS})
- new net SPI_MISO: U4.18 (IO20), U6.2 (DO(IO1))
- new net SPI_MOSI: U4.19 (IO21), U6.5 (DI(IO0))
- new net STATUS_LED: R17.1, TP4.1, U4.11 (IO10)
- new net USB_DN: J1.A7 (D-), J1.B7 (D-), TP6.1, U1.3 (I/O2), U1.4 (I/O2), U4.16 (IO18)
- new net USB_DP: J1.A6 (D+), J1.B6 (D+), TP5.1, U1.1 (I/O1), U1.6 (I/O1), U4.17 (IO19)
- new net VBAT_RAW: C3.1, J2.1 (Pin_1), SW1.1 (A), U2.5 (BAT)
- new net VBUS: C2.1, D3.2 (A), J1.A4 (VBUS), J1.A9 (VBUS), J1.B4 (VBUS), J1.B9 (VBUS), Q1.1 (G), R5.1, R6.1, R7.1, U1.5 (VBUS), U2.4 (VCC), U2.8 (CE)
